File: board/board.kicad_pcb (KiCad board)
At the start: 2 copper layers, 21 x 13 mm, 1 part

Commit message: initial commit
Parts:
- added C1: 1uF, Capacitor_SMD:C_0402_1005Metric, F.Cu at (146.6, 96.4)
- added C2: 10uF, Capacitor_SMD:C_1210_3225Metric, F.Cu at (146.7, 92.5)
- added C3: 33uF, Capacitor_SMD:C_1210_3225Metric, F.Cu at (153.2, 92.8)
- added C4: 33uF, Capacitor_SMD:C_1210_3225Metric, F.Cu at (153.2, 97.5)
- added C6: 100nF, Capacitor_SMD:C_0402_1005Metric, F.Cu at (146.6, 95.4)
- added FB1: 200R, 5A, Capacitor_SMD:C_0603_1608Metric, F.Cu at (157.3, 102.2)
- added FB2: 200R, 5A, Capacitor_SMD:C_0603_1608Metric, F.Cu at (156.3, 90.8)
- added J1: 022_battery_cells, on_edge:on_edge_2x05_device, F.Cu at (140.0, 96.5)
- added J2: 003_power, on_edge:on_edge_2x05_host, F.Cu at (161.0, 96.5)
- added L1: 744316100, TPS61022:744316100, F.Cu at (148.0, 100.1)
- added R1: 10k, Resistor_SMD:R_0603_1608Metric, F.Cu at (152.0, 101.5)
- added R2: 10k, Resistor_SMD:R_0603_1608Metric, F.Cu at (153.6, 101.5)
- added R3: 10k, Resistor_SMD:R_0603_1608Metric, F.Cu at (155.1, 101.5)
- added R4: 732k, Resistor_SMD:R_0603_1608Metric, F.Cu at (150.7, 93.3)
- added R5: 100k, Resistor_SMD:R_0603_1608Metric, F.Cu at (149.2, 93.3)
- added U1: ~, TPS61022:TPS61022, F.Cu at (150.1, 96.0)
- LOGO1: moved to B.Cu
- moved LOGO1 3.16 mm to (151.0, 96.0), turned to 180 degrees
Routing:
- net GND: track 0.00 -> 29.6 mm, vias 0 -> 40
- net /implementation/VOUT: track 0.00 -> 21.6 mm
- net /implementation/VIN: track 0.00 -> 12.8 mm
- net /implementation/MODE: track 0.00 -> 12.0 mm, vias 0 -> 2
- net Net-(J2-3.3V): track 0.00 -> 11.7 mm, vias 0 -> 1
- net /implementation/EN: track 0.00 -> 11.6 mm, vias 0 -> 2
- net /implementation/SW: track 0.00 -> 4.71 mm
- net /implementation/FB: track 0.00 -> 2.66 mm
- net Net-(J2-5V): track 0.00 -> 2.61 mm, vias 0 -> 1
- added copper zone on F.Cu, net /implementation/VIN
- added copper zone on B.Cu, net GND
- added copper zone on F.Cu, net GND
- added copper zone on In1.Cu, net GND
- added copper zone on In2.Cu, net GND
Other:
- outline, holes or cut-outs redrawn
- copper layers 2 -> 4
- board text added: "b140_v1.0 step_up_converter_TPS61022"
- board text added: "osf.003"
- board text added: "osf.022"
