File: board/implementation.kicad_sch (KiCad schematic)
At the start: 0 parts

Commit message: initial commit
Parts:
- added C1: 1uF, Capacitor_SMD:C_0402_1005Metric, symbol Device:C_Small
- added C2: 10uF, Capacitor_SMD:C_1210_3225Metric, symbol Device:C_Polarized_Small
- added C3, C4: 33uF, Capacitor_SMD:C_1210_3225Metric, symbol Device:C_Polarized_Small
- added C6: 100nF, Capacitor_SMD:C_0402_1005Metric, symbol Device:C_Small
- added L1: 744316100, TPS61022:744316100, symbol TPS61022:744316100
- added R1, R2, R3: 10k, Resistor_SMD:R_0603_1608Metric, symbol Device:R_Small
- added R4: 732k, Resistor_SMD:R_0603_1608Metric, symbol Device:R_Small
- added R5: 100k, Resistor_SMD:R_0603_1608Metric, symbol Device:R_Small
- added U1: ~, TPS61022:TPS61022, symbol TPS61022:TPS61022
Connections:
- net GND: now also C1.2, C2.2, C3.2, C4.2, C6.2, R3.2, R5.2, U1.1 (GND)
- new net EN: R1.2, U1.5 (EN)
- new net FB: R4.2, R5.1, U1.4 (FB)
- new net MODE: R2.2, R3.1, U1.6 (MODE)
- new net SW: L1.2, U1.2 (SW)
- new net VIN: C1.1, C2.1, C6.1, L1.1, R1.1, R2.1, U1.7 (VIN)
- new net VOUT: C3.1, C4.1, R4.1, U1.3 (VOUT)
Other:
- note added: "On off"
- note added: "PWM PFM"
- note added: "TPS61022 stepup"
